File: round_mote.sch (KiCad schematic (older format))
At the start: 34 parts, among them P1 RST-GND, P10 A5 A4, P11 GND RAW, P12 3.3V 5V, P2 D1 D0, P3 D3 D2, P4 D5 D4, P5 D9 D8, P6 D11 D10, P7 D13 D12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

Commit message: Upgraded KICAD to version 2011-03-30 BZR 2392
Parts:
- removed P6: D11 D10, symbol CONN_2
- added P6: D11 D10, symbol CONN_2

Commit message: Removed LED8 and added RX TX RSSI for Xbee
Parts:
- removed LEDA8: Green, SparkFun-LED-0603, symbol LED0603
- removed P10: A5 A4, symbol CONN_2
- removed RA3: 2.2k, SparkFun-0603-RES, symbol RESISTOR0603-RES
- added LEDX1: Red, SparkFun-LED-0603, symbol LED0603
- added LEDX2, LEDX3: Green, SparkFun-LED-0603, symbol LED0603
- added P10: A4 A5, symbol CONN_2
- added RX1, RX2, RX3: 2.2k, SparkFun-0603-RES, symbol RESISTOR0603-RES
- P5: value D9 D8 -> D8 D9
- P6: value D11 D10 -> D10 D11
- P7: value D13 D12 -> D12 D13
- P8: value A1 A0 -> A0 A1
- P9: value A3 A2 -> A2 A3
- R51, RA2: value 2.2k -> 4.7k
- renumbered P12 to P11, P11 to P12
Connections:
- net +3.3V: now also RX1.1, RX2.1; no longer U2.1 (VDD)
- net A4: now also P10.1 (P1)
- net A5: now also P10.2 (PM)
- net DIN: now also LEDX2.C
- net DOUT: now also LEDX1.C; no longer U2.2 (DOUT)
- net GND: now also LEDX3.C; no longer U2.10 (GND)
- net RSSI: now reaches U2.6 (RSSI)
- net RSSI: now also RX3.1
- new net: LEDX1.A, RX1.2
- new net: LEDX2.A, RX2.2
- new net: LEDX3.A, RX3.2
Other:
- moved on the sheet: DX1, DX2, P11, P12, U2
