File: round_mote.sch (KiCad schematic (older format))
At the start: 38 parts, among them P1 RST-GND, P10 A4 A5, P11 3.3V 5V, P12 GND RAW, P2 D1 D0, P3 D3 D2, P4 D5 D4, P5 D8 D9, P6 D10 D11, P7 D12 D13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

Commit message: added new logic level for xbee
Parts:
- removed DX1, DX2: DIODESOD, SparkFun-SOD-323, symbol DIODESOD
- added Q1, Q2, Q3: MOS_N, ~, symbol MOS_N
- added R1, R2, R3, R4, R5, R6: 1k, SparkFun-0603-RES, symbol RESISTOR0603-RES
- RX1, RX2, RX3: value 2.2k -> 1k
Connections:
- net +3.3V: now also Q1.1 (G), Q2.1 (G), Q3.1 (G), R1.1, R3.1, R5.1
- net +5V: now also R2.1, R4.1, R6.1
- net D8: now also Q3.3 (D), R6.2
- net DIN: now also U2.3 (DIN), Q2.2 (S), R3.2; no longer U1.11 (PD7(AIN1))
- net DOUT: now also Q1.2 (S), R1.2; no longer U1.10 (PD6(AIN0))
- net x9: now reaches U2.9 (DTR)
- net x9: now also Q3.2 (S), R5.2
- new net D6: Q1.3 (D), R2.2, U1.10 (PD6(AIN0))
- new net D7: Q2.3 (D), R4.2, U1.11 (PD7(AIN1))
